File: Switch-Board/Switch-Board.kicad_sch (KiCad schematic)
At the start: 21 parts, among them J1 Conn_01x08_Pin, J2 Conn_01x08_Pin, J3 Conn_01x08_Pin, J4 Conn_01x08_Pin, J5 Conn_01x01_Pin, SW1 SW_Nidec_CAS-120A1, SW10 SW_Nidec_CAS-120A1, SW11 SW_Nidec_CAS-120A1, SW12 SW_Nidec_CAS-120A1, SW13 SW_Nidec_CAS-120A1, SW14 SW_Nidec_CAS-120A1, SW15 SW_Nidec_CAS-120A1, SW16 SW_Nidec_CAS-120A1, SW2 SW_Nidec_CAS-120A1, SW3 SW_Nidec_CAS-120A1, SW4 SW_Nidec_CAS-120A1, SW5 SW_Nidec_CAS-120A1, SW6 SW_Nidec_CAS-120A1, SW7 SW_Nidec_CAS-120A1, SW8 SW_Nidec_CAS-120A1, SW9 SW_Nidec_CAS-120A1

Commit message: Finished Switch Board
Parts:
- added J10, J11, J12, J13, J14: Conn_01x01_Pin, Connector_Pin:Pin_D1.4mm_L8.5mm_W2.8mm_FlatFork, symbol Connector:Conn_01x01_Pin
- added J15, J16: Conn_01x01_Pin, MountingHole:MountingHole_2.5mm_Pad, symbol Connector:Conn_01x01_Pin
- added J17, J18, J19, J20: Conn_01x01_Pin, MountingHole:MountingHole_3.2mm_M3_DIN965_Pad, symbol Connector:Conn_01x01_Pin
- added J6, J7, J8, J9: Conn_01x01_Pin, Connector_Pin:Pin_D1.0mm_L10.0mm_LooseFit, symbol Connector:Conn_01x01_Pin
- J2, J4: footprint Connector_PinSocket_2.54mm:PinSocket_2x04_P2.54mm_Vertical -> Connector_PinHeader_2.54mm:PinHeader_1x08_P2.54mm_Vertical
- J5: footprint (none) -> Connector_Pin:Pin_D1.0mm_L10.0mm_LooseFit
Connections:
- net +5V: now also J15.1 (Pin_1), J6.1 (Pin_1), J7.1 (Pin_1), J8.1 (Pin_1), J9.1 (Pin_1)
- net at J1.8 (Pin_8), J2.8 (Pin_8): now also SW1.1 (C); no longer SW8.1 (C)
- net at J3.1 (Pin_1), J4.1 (Pin_1): now also SW16.3 (A); no longer SW9.1 (C)
- net at J3.2 (Pin_2), J4.2 (Pin_2): now also SW15.1 (C); no longer SW10.1 (C)
- net at J3.3 (Pin_3), J4.3 (Pin_3): now also SW14.1 (C); no longer SW11.1 (C)
- net at J3.4 (Pin_4), J4.4 (Pin_4): now also SW13.1 (C); no longer SW12.1 (C)
- net at J3.5 (Pin_5), J4.5 (Pin_5): now also SW12.1 (C); no longer SW13.1 (C)
- net at J3.6 (Pin_6), J4.6 (Pin_6): now also SW11.1 (C); no longer SW14.1 (C)
- net at J3.7 (Pin_7), J4.7 (Pin_7): now also SW10.1 (C); no longer SW15.1 (C)
- net at J3.8 (Pin_8), J4.8 (Pin_8): now also SW9.1 (C); no longer SW16.3 (A)
- net at J1.2 (Pin_2), J2.2 (Pin_2): now also SW7.1 (C); no longer SW2.1 (C)
- net at J1.1 (Pin_1), J2.1 (Pin_1): now also SW8.1 (C); no longer SW1.1 (C)
- net at J1.3 (Pin_3), J2.3 (Pin_3): now also SW6.1 (C); no longer SW3.1 (C)
- net at J1.4 (Pin_4), J2.4 (Pin_4): now also SW5.1 (C); no longer SW4.1 (C)
- net at J1.5 (Pin_5), J2.5 (Pin_5): now also SW4.1 (C); no longer SW5.1 (C)
- net at J1.6 (Pin_6), J2.6 (Pin_6): now also SW3.1 (C); no longer SW6.1 (C)
- net at J1.7 (Pin_7), J2.7 (Pin_7): now also SW2.1 (C); no longer SW7.1 (C)
- new net GND: J10.1 (Pin_1), J11.1 (Pin_1), J12.1 (Pin_1), J13.1 (Pin_1), J14.1 (Pin_1), J16.1 (Pin_1)
Other:
- moved on the sheet: J1, J2, J3, J4
